File: Prime_Maxel-v3.kicad_pcb (KiCad board)
At the start: 4 copper layers, 205 x 150 mm, 150 parts, among them J1 EJ503A, J2 PWM, J3 Power, J4 Analog, J5 PWM, J6 Analog, J7 Communication, J8 Digital, U1 TCA9548APWR, U10 LM324DRE4, U11 SLG47004V, U12 LM324DRE4, U13 SLG47004V, U14 LM324DRE4, U15 SLG47004V, U16 LM324DRE4, U17 SLG47004V, U18 LM324DRE4, U19 SLG47004V, U2 LM324DRE4, U20 LM324DRE4, U21 SLG47004V, U22 LM324DRE4, U23 SLG47004V, U24 LM324DRE4, U25 SLG47004V, U3 SLG47004V, U4 LM324DRE4, U5 SLG47004V, U6 LM324DRE4, U7 SLG47004V, U8 LM324DRE4, U9 SLG47004V

Commit message: v3 complete: experimental results published (Zenodo DOI 10.5281/zenodo.20637347)
- Rewrite README: completed research platform with published results
- Add Arduino sketches for all 15 frequency set experiments
- Add Python analysis pipeline (capture, FFT, experiment suite)
- Add research write-ups and published paper PDF
- Add LTspice simulations and GreenPAK configs
- Update license: CERN-OHL-S v2 (hardware) + Apache 2.0 (code)
- Clean .gitignore: exclude large/generated/personal files
Parts:
- turned U13 to 75 degrees
- turned U25 to -105 degrees
Routing:
- net GND_PWT: track 0.00 -> 131.4 mm, vias 0 -> 72
- net +VCC_PWT: track 0.00 -> 81.3 mm, vias 0 -> 60
- net /Golden Cell/TORSION_A: track 630.6 -> 646.6 mm
